File: kicad_src/PCB-SS.kicad_pcb (KiCad board)
At the start: 2 copper layers, 57.2 x 57.2 mm, 46 parts, among them J101 BATTERY_CONNECTOR, J102 SEESAW_I2C, J103 MSP_CONNECTOR_LEFT, J104 SCD30_BUS, J105 Conn_01x03_Male, J106 SEESAW_POWER, J107 LORA_BUS, J108 DPS310_BUS, Q101 FQP27P06, Q102 FQP27P06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

Commit message: Update PCB
Parts:
- removed C108: 22uF, Capacitor_SMD:C_0805_2012Metric
- removed L104: 2.2uH, NRH2412T2R2MNGH:NRH2412T2R2MNGH
- removed Q102, Q107: FQP27P06, digikey-footprints:TO-220-3
- removed R103: 10K, Resistor_SMD:R_0805_2012Metric
- removed R111, R116: 1K, Resistor_SMD:R_0805_2012Metric
- removed R114: 100K, Resistor_SMD:R_0805_2012Metric
- removed U104: LM3671MF-3.3, LM3671MF-3:SOT95P280X145-5N
- Q101, Q104, Q106: moved to B.Cu
- moved C104 36.8 mm to (140.6, 87.0)
- moved Q104 29.6 mm to (171.1, 103.0)
- moved Q106 24.5 mm to (171.1, 92.3)
- moved R110 16.5 mm to (163.0, 92.3)
- moved Q101 11.9 mm to (171.1, 113.9)
- moved C107 8.12 mm to (158.4, 77.2), turned to 90 degrees
- moved R104 7.91 mm to (162.1, 109.9), turned to 0 degrees
- moved C103 7.61 mm to (160.9, 84.5), turned to 270 degrees
- moved J105 5.36 mm to (171.1, 118.5)
- moved R113 4.13 mm to (163.2, 80.7), turned to 270 degrees
- moved L103 3.37 mm to (155.6, 80.7), turned to 90 degrees
- moved U103 3.37 mm to (159.7, 80.6)
Connections:
- net /SEESAW_5V_EN renamed /SENSORS_5V_EN
- C104 pad 1: Net-(C104-Pad1) -> VCC
- C107 pad 1: SEESAW_V_IN -> SENSORS_V_IN
- J103 pad 11: SEESAW_GPIO_EN -> Net-(J103-Pad11)
- J103 pad 13: SCD30_GPIO_EN -> Net-(J103-Pad13)
- J103 pad 9: DPS310_GPIO_EN -> SENSORS_GPIO_EN
- J104 pad 1: SCD30_V_IN -> SENSORS_V_IN
- J106 pad 1: SEESAW_V_IN -> SENSORS_V_IN
- J106 pad 3: SEESAW_V_IN -> SENSORS_V_IN
- J106 pad 5: SEESAW_V_IN -> SENSORS_V_IN
- J106 pad 7: SEESAW_V_IN -> SENSORS_V_IN
- J108 pad 1: DPS310_V_IN -> SENSORS_V_IN
- L103 pad 2: SEESAW_V_IN -> SENSORS_V_IN
- Q101 pad 2: +5V -> Net-(J105-Pad2)
- Q101 pad 3: Net-(J105-Pad2) -> +5V
- Q104 pad 2: +5V -> Net-(C102-Pad1)
- Q104 pad 3: Net-(C102-Pad1) -> +5V
- Q106 pad 2: +5V -> Net-(C103-Pad1)
- Q106 pad 3: Net-(C103-Pad1) -> +5V
- U103 pad 4: SEESAW_V_IN -> SENSORS_V_IN
- U106 pad 11: /SCD30_5V_EN -> Net-(U106-Pad11)
- U106 pad 3: SEESAW_GPIO_EN -> SENSORS_GPIO_EN
- U106 pad 4: SCD30_GPIO_EN -> Net-(U106-Pad4)
- U106 pad 8: Net-(R103-Pad2) -> +3V3
Routing:
- net SCD30_GPIO_EN: track 84.3 -> 0.00 mm, vias 9 -> 0
- net SENSORS_V_IN: track 0.00 -> 72.8 mm, vias 0 -> 3
- net DPS310_GPIO_EN: track 60.0 -> 0.00 mm, vias 3 -> 0
- net SEESAW_GPIO_EN: track 55.0 -> 0.00 mm, vias 5 -> 0
- net SENSORS_GPIO_EN: track 0.00 -> 52.4 mm, vias 0 -> 5
- net /SCD30_5V_EN: track 33.9 -> 0.00 mm, vias 3 -> 0
- net SEESAW_V_IN: track 31.6 -> 0.00 mm, vias 4 -> 0
- net Net-(C102-Pad1): track 11.0 -> 37.4 mm, vias 0 -> 1
- net +5V: track 170.0 -> 145.1 mm, vias 14 -> 13
- net SCD30_V_IN: track 23.0 -> 0.00 mm, vias 1 -> 0
- net /LORA_5V_EN: track 25.8 -> 45.1 mm, vias 2 -> 3
- net /SENSORS_5V_EN: track 36.0 -> 19.8 mm
- net DPS310_V_IN: track 15.1 -> 0.00 mm
- net Net-(R103-Pad2): track 11.9 -> 0.00 mm
- net Net-(C104-Pad1): track 9.02 -> 0.00 mm
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