File: kicad_src/PCB-SS.sch (KiCad schematic (older format))
At the start: 46 parts, among them J101 BATTERY_CONNECTOR, J102 SEESAW_I2C, J103 MSP_CONNECTOR_LEFT, J104 SCD30_BUS, J105 Conn_01x03_Male, J106 SEESAW_POWER, J107 LORA_BUS, J108 DPS310_BUS, Q101 FQP27P06, Q102 FQP27P06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

Commit message: Update PCB
Parts:
- removed C108: 22uF, Capacitor_SMD:C_0805_2012Metric, symbol Device:C
- removed L104: 2.2uH, NRH2412T2R2MNGH:NRH2412T2R2MNGH, symbol Device:L
- removed Q102, Q107: FQP27P06, digikey-footprints:TO-220-3, symbol dk_Transistors-FETs-MOSFETs-Single:FQP27P06
- removed R103: 10K, Resistor_SMD:R_0805_2012Metric, symbol Device:R_US
- removed R111, R116: 1K, Resistor_SMD:R_0805_2012Metric, symbol Device:R_US
- removed R114: 100K, Resistor_SMD:R_0805_2012Metric, symbol Device:R_US
- removed U104: LM3671MF-3.3, LM3671MF-3:SOT95P280X145-5N, symbol LM3671MF-3.3:LM3671MF-3.3
- J105: value Conn_01x03_Male -> SERVO_BUS
Connections:
- net SCD30_V_IN is gone; now on net SENSORS_V_IN: J104.1 (Pin_1)
- net SEESAW_V_IN is gone; now on net SENSORS_V_IN: C107.1, J106.1 (Pin_1), J106.3 (Pin_3), J106.5 (Pin_5), J106.7 (Pin_7), L103.2, U103.4 (FB)
- net +3V3: now also U106.8 (OE)
- net +5V: now also Q101.3 (S), Q104.3 (S), Q106.3 (S); no longer Q101.2 (D), Q104.2 (D), Q106.2 (D)
- net VCC: now also C104.1
- net at C102.1, R112.2, U102.1 (VIN): now also Q104.2 (D); no longer Q104.3 (S)
- net at C103.1, R113.2, U103.1 (VIN): now also Q106.2 (D); no longer Q106.3 (S)
- net at J105.2 (Pin_2): now also Q101.2 (D); no longer Q101.3 (S)
- net DPS310_GPIO_EN renamed SENSORS_GPIO_EN
- net SENSORS_GPIO_EN: now also U106.3 (A0)
- net DPS310_V_IN renamed SENSORS_V_IN
- net SCD30_5V_EN: no longer names the net of U106.11 (B1)
- net SCD30_GPIO_EN: no longer names the net of J103.13 (Pin_13)
- net SCD30_GPIO_EN: no longer U106.4 (A1)
- net SEESAW_5V_EN renamed SENSORS_5V_EN
- net SEESAW_GPIO_EN: no longer names the net of J103.11 (Pin_11)
- net SEESAW_GPIO_EN: no longer U106.3 (A0)
- no-connect marks 10 -> 12
Other:
- moved on the sheet: C102, C103, C105, C106, C107, C110, J105, L101, L102, L103, Q101, Q104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
